File: docs/Kicad/RFBoat.kicad_sch (KiCad schematic)
At the start: 12 parts, among them SW1 SW_DPST, U1 L293D, U2 5V regulator, U3 NRF24L01_Breakout

Commit message: changed pin layout to free last PWM pin (10) CE & CSN
Parts:
- added BAUX1: (no value), symbol Device:Battery
- added R1: (no value), symbol Device:R_Photo
- added R2: (no value), symbol Device:R
- added SERV1: (no value), symbol Motor:Motor_Servo
- BTMOT1: footprint (none) -> Connector_JST:JST_PH_B2B-PH-K_1x02_P2.00mm_Vertical
- C2, C3: value (none) -> C; footprint (none) -> Capacitor_THT:C_Disc_D3.4mm_W2.1mm_P2.50mm
- M.STD2: value (none) -> Starboard
Connections:
- net at U3.3 (CE): now also A1.11 (D8); no longer A1.13 (D10)
- net at U3.4 (~{CSN}): now also A1.10 (D7); no longer A1.12 (D9)
- net at A1.27 (+5V), U1.16 (VCC1), U2.3 (VO): now also R1.1
- net at U1.15 (4A): now also A1.12 (D9); no longer A1.10 (D7)
- net at A1.19 (A0): now also R1.2, R2.1
- net at A1.29 (GND): now also BAUX1.2 (-), R2.2, SERV1.3 (-)
- new net: BAUX1.1 (+), SERV1.2 (+)
- new net: A1.13 (D10), SERV1.1 (PWM)
- no-connect marks 17 -> 14
Other:
- moved on the sheet: A1, C1
